Commit message: Fixed references to hexapodo_description package

File: clhero_sim_description/urdf/base.robot.xacro (robot description, xacro)
@@ -34,5 +34,5 @@
         <origin xyz="${0/1e3} 0 0" rpy="${pi/2} 0 0"/>
         <geometry>
-            <mesh filename="package://hexapodo_description/meshes/chassis_piezas.stl" scale="0.01 0.01 0.01"/>
+            <mesh filename="package://clhero_sim_description/meshes/chassis_piezas.stl" scale="0.01 0.01 0.01"/>
         </geometry>
         <material name="base_link_material">
@@ -43,5 +43,5 @@
         <origin xyz="${0/1e3} 0 0" rpy="${pi/2} 0 0"/>
         <geometry>
-            <mesh filename="package://hexapodo_description/meshes/chassis_piezas.stl" scale="0.01 0.01 0.01"/>
+            <mesh filename="package://clhero_sim_description/meshes/chassis_piezas.stl" scale="0.01 0.01 0.01"/>
         </geometry>
     </collision>

File: clhero_sim_description/urdf/base.xacro (robot description, xacro)
@@ -35,5 +35,5 @@
         <origin xyz="${-300/1e3} 0 0" rpy="${pi/2} 0 ${pi/2}"/>
         <geometry>
-            <mesh filename="package://hexapodo_description/meshes/chassis.stl" scale="0.001 0.001 0.001"/>
+            <mesh filename="package://clhero_sim_description/meshes/chassis.stl" scale="0.001 0.001 0.001"/>
         </geometry>
         <material name="base_link_material">
@@ -44,5 +44,5 @@
         <origin xyz="${-300/1e3} 0 0" rpy="${pi/2} 0 ${pi/2}"/>
         <geometry>
-            <mesh filename="package://hexapodo_description/meshes/chassis.stl" scale="0.001 0.001 0.001"/>
+            <mesh filename="package://clhero_sim_description/meshes/chassis.stl" scale="0.001 0.001 0.001"/>
         </geometry>
     </collision>

File: clhero_sim_description/urdf/base_cinta.xacro (robot description, xacro)
@@ -29,5 +29,5 @@
         <origin xyz="0 0 0.38" rpy="0 0 ${pi/2}"/>
         <geometry>
-            <mesh filename="package://hexapodo_description/meshes/cinta_barreras.stl" scale="0.01 0.01 0.01"/>
+            <mesh filename="package://clhero_sim_description/meshes/cinta_barreras.stl" scale="0.01 0.01 0.01"/>
         </geometry>
         <material name="base_link_material">
@@ -44,5 +44,5 @@
         <origin xyz="0 0 0.358" rpy="0 0 0"/>
         <geometry>
-            <mesh filename="package://hexapodo_description/meshes/cinta_barreras.stl" scale="0.01 0.01 0.01"/>
+            <mesh filename="package://clhero_sim_description/meshes/cinta_barreras.stl" scale="0.01 0.01 0.01"/>
         </geometry>
     </collision-->
@@ -65,5 +65,5 @@
         <origin xyz="${-300/1e3} 0 0.0" rpy="${pi/2} 0 ${pi/2}"/>
         <geometry>
-            <mesh filename="package://hexapodo_description/meshes/chassis.stl" scale="0.001 0.001 0.001"/>
+            <mesh filename="package://clhero_sim_description/meshes/chassis.stl" scale="0.001 0.001 0.001"/>
         </geometry>
         <material name="chassis_material">
@@ -74,5 +74,5 @@
         <origin xyz="${-300/1e3} 0 0.0" rpy="${pi/2} 0 ${pi/2}"/>
         <geometry>
-            <mesh filename="package://hexapodo_description/meshes/chassis.stl" scale="0.001 0.001 0.001"/>
+            <mesh filename="package://clhero_sim_description/meshes/chassis.stl" scale="0.001 0.001 0.001"/>
         </geometry>
     </collision>

File: clhero_sim_description/urdf/base_locked.xacro (robot description, xacro)
@@ -42,5 +42,5 @@
         <origin xyz="0 0 0" rpy="${pi/2} 0 0"/>
         <geometry>
-            <mesh filename="package://hexapodo_description/meshes/chassis_piezas.stl" scale="0.01 0.01 0.01"/>
+            <mesh filename="package://clhero_sim_description/meshes/chassis_piezas.stl" scale="0.01 0.01 0.01"/>
         </geometry>
         <material name="base_link_material">
@@ -51,5 +51,5 @@
         <origin xyz="0 0 0" rpy="${pi/2} 0 0"/>
         <geometry>
-            <mesh filename="package://hexapodo_description/meshes/chassis_piezas.stl" scale="0.01 0.01 0.01"/>
+            <mesh filename="package://clhero_sim_description/meshes/chassis_piezas.stl" scale="0.01 0.01 0.01"/>
         </geometry>
     </collision>

File: clhero_sim_description/urdf/base_pedestal.xacro (robot description, xacro)
@@ -44,5 +44,5 @@
         <origin xyz="${-300/1e3} 0 0" rpy="${pi/2} 0 ${pi/2}"/>
         <geometry>
-            <mesh filename="package://hexapodo_description/meshes/chassis.stl" scale="0.001 0.001 0.001"/>
+            <mesh filename="package://clhero_sim_description/meshes/chassis.stl" scale="0.001 0.001 0.001"/>
         </geometry>
         <material name="base_link_material">
@@ -53,5 +53,5 @@
         <origin xyz="${-300/1e3} 0 0" rpy="${pi/2} 0 ${pi/2}"/>
         <geometry>
-            <mesh filename="package://hexapodo_description/meshes/chassis.stl" scale="0.001 0.001 0.001"/>
+            <mesh filename="package://clhero_sim_description/meshes/chassis.stl" scale="0.001 0.001 0.001"/>
         </geometry>
     </collision>

File: clhero_sim_description/urdf/pata_c.robot.xacro (robot description, xacro)
@@ -30,5 +30,5 @@
             </xacro:if>
             <geometry>
-                <mesh filename="package://hexapodo_description/meshes/pvc.stl" scale="0.001 0.001 0.001"/>
+                <mesh filename="package://clhero_sim_description/meshes/pvc.stl" scale="0.001 0.001 0.001"/>
             </geometry>
             <material name="Grey">
@@ -44,5 +44,5 @@
             </xacro:if>
             <geometry>
-                <mesh filename="package://hexapodo_description/meshes/pvc.stl" scale="0.001 0.001 0.001"/>
+                <mesh filename="package://clhero_sim_description/meshes/pvc.stl" scale="0.001 0.001 0.001"/>
             </geometry>
         </collision>

File: clhero_sim_description/urdf/pata_c.xacro (robot description, xacro)
@@ -36,5 +36,5 @@
             </xacro:if>
             <geometry>
-                <mesh filename="package://hexapodo_description/meshes/pvc.stl" scale="0.001 0.001 0.001"/>
+                <mesh filename="package://clhero_sim_description/meshes/pvc.stl" scale="0.001 0.001 0.001"/>
             </geometry>
             <material name="Grey">
@@ -50,5 +50,5 @@
             </xacro:if>
             <geometry>
-                <mesh filename="package://hexapodo_description/meshes/pvc.stl" scale="0.001 0.001 0.001"/>
+                <mesh filename="package://clhero_sim_description/meshes/pvc.stl" scale="0.001 0.001 0.001"/>
             </geometry>
             <surface>

File: clhero_sim_description/urdf/pata_c_cinta.xacro (robot description, xacro)
@@ -30,5 +30,5 @@
             </xacro:if>
             <geometry>
-                <mesh filename="package://hexapodo_description/meshes/pvc.stl" scale="0.001 0.001 0.001"/>
+                <mesh filename="package://clhero_sim_description/meshes/pvc.stl" scale="0.001 0.001 0.001"/>
             </geometry>
             <material name="Grey">
@@ -44,5 +44,5 @@
             </xacro:if>
             <geometry>
-                <mesh filename="package://hexapodo_description/meshes/pvc.stl" scale="0.001 0.001 0.001"/>
+                <mesh filename="package://clhero_sim_description/meshes/pvc.stl" scale="0.001 0.001 0.001"/>
             </geometry>
         </collision>

File: clhero_sim_description/urdf/pata_c_locked.xacro (robot description, xacro)
@@ -29,5 +29,5 @@
             </xacro:if>
             <geometry>
-                <mesh filename="package://hexapodo_description/meshes/pvc.stl" scale="0.001 0.001 0.001"/>
+                <mesh filename="package://clhero_sim_description/meshes/pvc.stl" scale="0.001 0.001 0.001"/>
             </geometry>
             <material name="Grey">
@@ -43,5 +43,5 @@
             </xacro:if>
             <geometry>
-                <mesh filename="package://hexapodo_description/meshes/pvc.stl" scale="0.001 0.001 0.001"/>
+                <mesh filename="package://clhero_sim_description/meshes/pvc.stl" scale="0.001 0.001 0.001"/>
             </geometry>
         </collision>
